File: Hardware/Shield_Esp32.kicad_pcb (KiCad board)
At the start: 2 copper layers, 43 parts, among them J1 Conn_01x02_Male, J10 Conn_01x02_Male, J11 Conn_01x02_Male, J12 Conn_01x02_Male, J13 Conn_01x02_Male, J14 Conn_01x02_Male, J15 Conn_01x02_Male, J16 Conn_01x02_Male, J17 Conn_01x02_Male, J18 Conn_01x02_Male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

Commit message: pcb att
Parts:
- moved D2 41.3 mm to (179.1, 82.3), turned to -90 degrees
- moved J2 41.0 mm to (179.2, 74.8)
- moved D7 35.0 mm to (121.8, 95.9), turned to -90 degrees
- moved D1 30.8 mm to (184.0, 82.3), turned to -90 degrees
- moved J23 30.6 mm to (124.3, 90.9), turned to 90 degrees
- moved J1 30.6 mm to (184.1, 74.8)
- moved D8 29.0 mm to (126.3, 95.9), turned to -90 degrees
- moved J3 19.0 mm to (133.5, 84.9)
- moved D3 19.0 mm to (122.5, 114.2)
- moved D4 19.0 mm to (124.9, 105.4)
- moved J7 19.0 mm to (124.1, 100.2)
- moved J8 19.0 mm to (126.8, 110.4)
- moved R1 19.0 mm to (126.7, 114.2)
- moved J6 18.8 mm to (124.2, 85.9)
- moved J15 3.34 mm to (166.5, 67.0)
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Routing:
- net +3.3V: track 0.00 -> 186.0 mm, vias 0 -> 5
- net +5V: track 0.00 -> 104.1 mm, vias 0 -> 2
- net GND: track 0.00 -> 103.0 mm, vias 0 -> 4
- net ENC0: track 0.00 -> 91.0 mm
- net RXB: track 0.00 -> 81.3 mm, vias 0 -> 1
- net PWM1N: track 0.00 -> 77.9 mm
- net TXB: track 0.00 -> 76.2 mm, vias 0 -> 1
- net ADC0: track 0.00 -> 72.6 mm
- net ADC1: track 0.00 -> 67.3 mm
- net PWM1: track 0.00 -> 59.7 mm
- net R_TCRT: track 0.00 -> 53.7 mm
- net TRIG0: track 0.00 -> 50.3 mm
- net PWM2N: track 0.00 -> 50.0 mm
- net L_TCRT: track 0.00 -> 49.9 mm
- net ECHO0: track 0.00 -> 44.8 mm
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- added copper zone on B.Cu, net GND
- added copper zone on F.Cu, net GND
Other:
- board outline added: 93 x 70.5 mm

Commit message: pcb update
Parts:
- C1, C2, D1, D2, D4, D5, D6, D7, D8, R2, R3, R4, R5, R6, R7, R8, R9: moved to B.Cu
- moved J23 40.2 mm to (151.9, 120.1), turned to 180 degrees
- moved D3 37.7 mm to (137.9, 79.8), turned to 90 degrees
- moved R1 37.2 mm to (140.5, 79.7), turned to 90 degrees
- moved J7 36.6 mm to (156.3, 117.5), turned to 0 degrees
- moved D7 35.8 mm to (147.2, 121.0), turned to 0 degrees
- moved J8 31.7 mm to (129.3, 78.8), turned to 90 degrees
- moved D8 29.7 mm to (147.2, 117.0)
- moved J6 28.3 mm to (152.3, 82.1), turned to 180 degrees
- moved D4 28.3 mm to (139.2, 81.0), turned to -90 degrees
- moved J15 12.7 mm to (164.5, 79.5)
- moved J17 12.6 mm to (172.5, 79.5)
- moved D5 10.3 mm to (187.3, 108.1), turned to -90 degrees
- moved D6 10.2 mm to (183.0, 108.0), turned to -90 degrees
- moved D1 9.75 mm to (182.5, 91.9), turned to 90 degrees
- moved D2 9.66 mm to (178.0, 91.9), turned to 90 degrees
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Routing:
- net AMP2: track 6.86 -> 156.0 mm, vias 0 -> 1
- net GND: track 103.0 -> 13.3 mm, vias 4 -> 6
- net +5V: track 104.1 -> 36.6 mm, vias 2 -> 0
- net +3.3V: track 186.0 -> 132.3 mm, vias 5 -> 0
- net ADC2: track 17.7 -> 71.3 mm
- net L_TCRT: track 49.9 -> 98.2 mm
- net ADC3: track 15.2 -> 60.2 mm, vias 0 -> 1
- net ENC0: track 91.0 -> 52.5 mm, vias 0 -> 1
- net ADC1: track 67.3 -> 103.9 mm
- net +5VP: track 11.3 -> 37.8 mm
- net TXB: track 76.2 -> 100.5 mm, vias 1 -> 0
- net AMP1: track 7.35 -> 30.8 mm
- net D26: track 21.3 -> 9.03 mm
- net D14: track 21.3 -> 9.43 mm
- net TX0: track 17.9 -> 10.3 mm
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Other:
- board size 93 x 70.5 mm -> 79.9 x 52 mm

Commit message: pcb update
Parts:
- moved D7 65.8 mm to (198.2, 79.4), turned to 180 degrees
- moved D8 61.0 mm to (198.2, 83.4), turned to 90 degrees
- moved J12 59.3 mm to (150.6, 80.5), turned to 0 degrees
- moved J23 57.6 mm to (193.5, 80.3), turned to 0 degrees
- moved J6 54.6 mm to (193.1, 118.3), turned to 0 degrees
- moved J21 53.4 mm to (154.8, 80.4), turned to 0 degrees
- moved J9 52.6 mm to (188.9, 120.9), turned to 180 degrees
- moved J10 48.0 mm to (184.9, 120.9), turned to 180 degrees
- moved J1 47.7 mm to (160.8, 120.9), turned to 180 degrees
- moved J7 47.7 mm to (189.1, 82.9), turned to 180 degrees
- moved J19 46.3 mm to (184.7, 80.4), turned to 0 degrees
- moved J4 46.1 mm to (153.6, 113.1), turned to 90 degrees
- moved J5 45.7 mm to (153.6, 87.7), turned to 90 degrees
- moved J15 44.5 mm to (180.9, 120.9), turned to 180 degrees
- moved J2 44.2 mm to (164.9, 120.9), turned to 180 degrees
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Routing:
- net PWM2: track 46.1 -> 133.4 mm
- net AMP1: track 30.8 -> 108.4 mm
- net AMP2: track 156.0 -> 96.8 mm
- net L_TCRT: track 98.2 -> 45.1 mm
- net ADC3: track 60.2 -> 107.5 mm
- net ECHO1: track 39.3 -> 84.8 mm
- net +5V: track 36.6 -> 80.7 mm, vias 0 -> 1
- net TRIG1: track 46.0 -> 84.9 mm, vias 1 -> 0
- net ADC1: track 103.9 -> 69.9 mm
- net ADC2: track 71.3 -> 102.8 mm, vias 1 -> 0
- net ENC1: track 44.1 -> 74.7 mm
- net TXB: track 100.5 -> 79.0 mm
- net PWM2N: track 47.9 -> 66.8 mm
- net ENC0: track 52.5 -> 71.4 mm, vias 1 -> 0
- net ECHO0: track 43.7 -> 62.4 mm, vias 1 -> 0
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Other:
- board size 79.9 x 52 mm -> 81.9 x 53.8 mm

Commit message: pcb update + new pcb
Parts:
- moved J8 79.0 mm to (202.8, 107.8), turned to 0 degrees
- moved D3 73.0 mm to (199.3, 119.3)
- moved R1 68.9 mm to (196.9, 119.3)
- moved D4 61.1 mm to (194.2, 107.7), turned to 90 degrees
- moved J3 7.32 mm to (137.7, 88.3)
- moved J11 4.42 mm to (159.2, 79.2), turned to 90 degrees
- moved J12 3.17 mm to (152.0, 83.3), turned to 90 degrees
- moved J21 3.03 mm to (152.0, 79.2), turned to 90 degrees
- moved J16 1.93 mm to (175.0, 120.5)
- moved J6 1.93 mm to (191.2, 118.0)
- moved J9 1.93 mm to (187.0, 120.5)
- moved J1 1.93 mm to (158.9, 120.5)
- moved J10 1.93 mm to (183.0, 120.5)
- moved J15 1.93 mm to (179.0, 120.5)
- moved J17 1.93 mm to (171.0, 120.5)
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Routing:
- net +5V: track 80.7 -> 24.4 mm
- net ADC0: track 61.7 -> 112.9 mm
- net ENC1: track 74.7 -> 111.7 mm
- net +5VP: track 27.5 -> 58.5 mm, vias 0 -> 2
- net TRIG1: track 84.9 -> 56.9 mm, vias 0 -> 2
- net +3.3V: track 131.6 -> 104.8 mm, vias 4 -> 0
- net PWM2N: track 66.8 -> 92.4 mm
- net ADC3: track 107.5 -> 83.9 mm, vias 1 -> 2
- net AMP1: track 108.4 -> 85.9 mm, vias 0 -> 2
- net RXB: track 72.4 -> 54.9 mm
- net ADC2: track 102.8 -> 87.3 mm, vias 0 -> 2
- net PWM2: track 133.4 -> 118.2 mm, vias 0 -> 2
- net ADC1: track 69.9 -> 84.0 mm
- net TXB: track 79.0 -> 66.5 mm, vias 0 -> 2
- net PWM1: track 80.9 -> 69.0 mm, vias 1 -> 0
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Other:
- board size 81.9 x 53.8 mm -> 81.3 x 55.3 mm

Commit message: final pcb
Routing:
- net GND: track 5.91 -> 13.5 mm
Changed lines of the file:
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@@
   (segment (start 189.16 113.075) (end 189.16 111.1859) (width 0.762) (layer "B.Cu") (net 1))
   (segment (start 199.4618 112.84) (end 202.8 112.84) (width 0.762) (layer "B.Cu") (net 1))
-  (segment (start 194.2 109.8) (end 192.1609 109.8) (width 0.762) (layer "B.Cu") (net 1))
   (segment (start 196.2391 109.8) (end 199.2791 112.84) (width 0.762) (layer "B.Cu") (net 1))
   (segment (start 195.2196 109.8) (end 196.2391 109.8) (width 0.762) (layer "B.Cu") (net 1))
-  (segment (start 192.1609 109.8) (end 191.9609 109.6) (width 0.762) (layer "B.Cu") (net 1))
+  (segment (start 194.2 109.8) (end 189.1 109.8) (width 0.762) (layer "B.Cu") (net 1))
   (segment (start 188.9 110.9259) (end 189.16 111.1859) (width 0.762) (layer "B.Cu") (net 1))
   (segment (start 199.4618 112.84) (end 199.4618 116.3961) (width 0.762) (layer "B.Cu") (net 1))
-  (segment (start 191.9609 109.6) (end 188.9 109.6) (width 0.762) (layer "B.Cu") (net 1))
+  (segment (start 189.1 109.8) (end 188.9 109.6) (width 0.762) (layer "B.Cu") (net 1))
   (segment (start 188.9 109.6) (end 188.9 110.9259) (width 0.762) (layer "B.Cu") (net 1))
   (segment (start 199.2791 112.84) (end 199.4618 112.84) (width 0.762) (layer "B.Cu") (net 1))
@@
   (via (at 160.2795 91.4338) (size 1.8) (drill 0.6) (layers "F.Cu" "B.Cu") (net 2))
   (via (at 200.5928 77.1072) (size 1.8) (drill 0.6) (layers "F.Cu" "B.Cu") (net 2))
+  (segment (start 171.4 107.8875) (end 173.8875 107.8875) (width 0.762) (layer "B.Cu") (net 2))
+  (segment (start 178.7416 108.0584) (end 178.9 107.9) (width 0.762) (layer "B.Cu") (net 2))
+  (segment (start 186.62 113.075) (end 186.62 109.805) (width 0.762) (layer "B.Cu") (net 2))
+  (segment (start 173.9 107.9) (end 174.0584 108.0584) (width 0.762) (layer "B.Cu") (net 2))
+  (segment (start 160.2795 92.0455) (end 159.05 93.275) (width 0.762) (layer "B.Cu") (net 2))
+  (segment (start 173.8875 107.8875) (end 173.9 107.9) (width 0.762) (layer "B.Cu") (net 2))
+  (segment (start 160.2795 91.4338) (end 160.2795 92.0455) (width 0.762) (layer "B.Cu") (net 2))
+  (segment (start 174.0584 108.0584) (end 178.7416 108.0584) (width 0.762) (layer "B.Cu") (net 2))
   (segment (start 186.62 109.805) (end 186.825 109.6) (width 0.762) (layer "B.Cu") (net 2))
-  (segment (start 160.2795 92.0455) (end 159.05 93.275) (width 0.762) (layer "B.Cu") (net 2))
-  (segment (start 186.62 113.075) (end 186.62 109.805) (width 0.762) (layer "B.Cu") (net 2))
-  (segment (start 160.2795 91.4338) (end 160.2795 92.0455) (width 0.762) (layer "B.Cu") (net 2))
   (segment (start 200.7 80.5) (end 199.1 80.5) (width 0.762) (layer "B.Cu") (net 3))
   (segment (start 163.85 104.7401) (end 163.85 107.525) (width 0.762) (layer "B.Cu") (net 3))
@@
       )
     )
+  )
+  (zone (net 0) (net_name "") (layer "B.Cu") (hatch edge 0.508)
+    (connect_pads (clearance 0))
+    (min_thickness 0.254)
+    (keepout (tracks allowed) (vias allowed) (pads allowed ) (copperpour not_allowed) (footprints allowed))
+    (fill (thermal_gap 0.508) (thermal_bridge_width 0.508))
+    (polygon
+      (pts
+        (xy 174.4 107)
+        (xy 173.3 106.9)
+        (xy 173.3 106.7)
+        (xy 174.4 106.7)
+      )
+    )
+  )
+  (zone (net 0) (net_name "") (layer "B.Cu") (hatch edge 0.508)
+    (connect_pads (clearance 0))
+    (min_thickness 0.254)
+    (keepout (tracks allowed) (vias allowed) (pads allowed ) (copperpour not_allowed) (footprints allowed))
+    (fill (thermal_gap 0.508) (thermal_bridge_width 0.508))
+    (polygon
+      (pts
+        (xy 165.7 107.2)
+        (xy 164.6 107.1)
+        (xy 164.6 106.9)
+        (xy 165.7 106.9)
+      )
+    )
+  )
+  (zone (net 0) (net_name "") (layer "B.Cu") (hatch edge 0.508)
+    (connect_pads (clearance 0))
+    (min_thickness 0.254)
+    (keepout (tracks allowed) (vias allowed) (pads allowed ) (copperpour not_allowed) (footprints allowed))
+    (fill (thermal_gap 0.508) (thermal_bridge_width 0.508))
+    (polygon
+      (pts
+        (xy 170.5 107.3)
+        (xy 170.4 108.4)
+        (xy 170.2 108.4)
+        (xy 170.2 107.3)
+      )
+    )
+  )
+  (zone (net 0) (net_name "") (layer "B.Cu") (hatch edge 0.508)
+    (connect_pads (clearance 0))
+    (min_thickness 0.254)
+    (keepout (tracks allowed) (vias allowed) (pads allowed ) (copperpour not_allowed) (footprints allowed))
+    (fill (thermal_gap 0.508) (thermal_bridge_width 0.508))
+    (polygon
+      (pts
+        (xy 156.2 94.1)
+        (xy 155 94.1)
+        (xy 155.1 93.8)
+        (xy 156.2 93.8)
+      )
+    )
+  )
+  (zone (net 0) (net_name "") (layer "B.Cu") (hatch edge 0.508)
+    (connect_pads (clearance 0))
+    (min_thickness 0.254)
+    (keepout (tracks allowed) (vias allowed) (pads allowed ) (copperpour not_allowed) (footprints allowed))
+    (fill (thermal_gap 0.508) (thermal_bridge_width 0.508))
+    (polygon
+      (pts
+        (xy 171.9 107.1)
+        (xy 170.8 107)
+        (xy 170.8 106.8)
+        (xy 171.9 106.8)
+      )
+    )
+  )
+  (zone (net 0) (net_name "") (layer "B.Cu") (hatch edge 0.508)
+    (connect_pads (clearance 0))
+    (min_thickness 0.254)
+    (keepout (tracks allowed) (vias allowed) (pads allowed ) (copperpour not_allowed) (footprints allowed))
+    (fill (thermal_gap 0.508) (thermal_bridge_width 0.508))
+    (polygon
+      (pts
+        (xy 165.7 107.1)
+        (xy 165.6 108.2)
+        (xy 165.4 108.2)
+        (xy 165.4 107.1)
+      )
+    )

Commit message: pcb update
Parts:
- added H1: MountingHole, MountingHole:MountingHole_2.2mm_M2, F.Cu at (128.3, 124.0)
- added H2: MountingHole, MountingHole:MountingHole_2.2mm_M2, F.Cu at (128.3, 75.3)
- added H3: MountingHole, MountingHole:MountingHole_2.2mm_M2, F.Cu at (202.9, 75.2)
- moved R1 2.57 mm to (198.4, 121.4), turned to 0 degrees
- moved J6 2.55 mm to (191.0, 120.5), turned to 180 degrees
- moved D6 2.31 mm to (164.7, 92.6)
- moved D8 1.30 mm to (197.9, 84.7)
- moved D3 1.08 mm to (198.3, 118.8), turned to 0 degrees
- moved D7 0.95 mm to (198.1, 80.5)
- moved D5 0.88 mm to (158.9, 92.6)
- moved D2 0.60 mm to (168.0, 108.5)
- moved D1 0.38 mm to (163.2, 108.7), turned to 0 degrees
Routing:
- net ADC0: track 112.9 -> 69.8 mm
- net GND: track 13.5 -> 6.29 mm, vias 6 -> 8
- net +3.3V: track 104.8 -> 111.3 mm
- net ECHO1: track 94.4 -> 98.3 mm
- net L_TCRT: track 44.0 -> 47.5 mm
- net AMP1: track 85.9 -> 88.8 mm
- net ADC3: track 83.9 -> 86.4 mm
- net PWM2: track 118.2 -> 115.7 mm
- net +5V: track 24.4 -> 26.0 mm
- net ENC0: track 63.3 -> 61.7 mm
- net R_TCRT: track 51.0 -> 52.2 mm
- net RX0: track 8.84 -> 9.99 mm
- net PWM1: track 69.0 -> 69.7 mm
- net +5VP: track 58.5 -> 57.8 mm
- net RXB: track 54.9 -> 55.4 mm
Other:
- board text added: "3V"
- board text added: "5V"
- board text added: "ESP32 Buggy Shield"
- board text added: "GND"
- board text added: "Nycolas Abreu"
- board text added: "Power"
