File: Hardware/Shield_Esp32.kicad_sch (KiCad schematic)
At the start: 3 parts

Commit message: Update Shield_Esp32.kicad_sch
Parts:
- added D? (x4): BAT54S, Package_TO_SOT_SMD:SOT-23, symbol Diode:BAT54S
- added D?: D_Schottky, symbol Device:D_Schottky
- added J? (x14): Conn_01x02_Male, Connector_PinHeader_2.54mm:PinHeader_1x02_P2.54mm_Vertical, symbol Connector:Conn_01x02_Male
- added R? (x4): 15k, Resistor_SMD:R_0805_2012Metric, symbol Device:R
- added R? (x4): 10k, Resistor_SMD:R_0805_2012Metric, symbol Device:R
Connections:
- net +3.3V: now also D?.2, D?.2, D?.2, D?.2
- net +5V: now also D?.1 (K); no longer J?.15 (Pin_15), J?.16 (Pin_16)
- net ADC0: now also J?.1 (Pin_1)
- net ADC1: now also J?.1 (Pin_1)
- net D12: now also J?.2 (Pin_2)
- net D13: now also R?.1, R?.2
- net D14: now also R?.1, R?.2
- net D18: now also J?.2 (Pin_2)
- net D19: now also J?.2 (Pin_2)
- net D2: now also R?.1, R?.2
- net D21: now also J?.2 (Pin_2)
- net D22: now also J?.2 (Pin_2)
- net D27: now also J?.2 (Pin_2)
- net D34: now also D?.3, J?.2 (Pin_2)
- net D35: now also D?.3, J?.2 (Pin_2)
- net D4: now also R?.1, R?.2
- net ECHO1: now also J?.1 (Pin_1)
- net GND: now also D?.1, D?.1, D?.1, D?.1, R?.2, R?.2, R?.2, R?.2
- net PWM1: now also J?.1 (Pin_1)
- net PWM1N: now also J?.1 (Pin_1)
- net PWM2: now also J?.1 (Pin_1)
- net PWM2N: now also J?.1 (Pin_1)
- net RX0: now also D?.3, J?.2 (Pin_2)
- net RXB: now also J?.1 (Pin_1)
- net TRIG0: now also J?.1 (Pin_1)
- net TRIG1: now also J?.1 (Pin_1)
- net TX0: now also D?.3, J?.2 (Pin_2)
- net TXB: now also J?.1 (Pin_1)
- net D0 renamed ENC0
- net ENC0: now also J?.1 (Pin_1)
- net D1 renamed ENC1
- net ENC1: now also J?.1 (Pin_1)
- new net: J?.2 (Pin_2), R?.1 (x4)
- new net +5VP: D?.2 (A), J?.15 (Pin_15), J?.16 (Pin_16)
- new net ECH0: J?.1 (Pin_1)
Other:
- note added: "ENCODER"
- note added: "Ligação em software de D21 e D22 no mesmo canal D21 e D22 geram mesmo sinal PWM Ligação em software de D18 e D19 no mesmo canal D18 e D19 geram mesmo sinal PWM"
- note added: "PWM"
- note added: "UART"
- note added: "Ultrasonic sensor"
- company: IFSC - Florianópolis -> Nycolas Coelho de Abreu IFSC - Florianópolis

Commit message: Update Shield_Esp32.kicad_sch
Parts:
- added C1: 100n, symbol Device:C
- added D3: LED, LED_SMD:LED_0805_2012Metric, symbol Device:LED
- added J17, J18, J6, J7: Conn_01x02_Male, Connector_PinHeader_2.54mm:PinHeader_1x02_P2.54mm_Vertical, symbol Connector:Conn_01x02_Male
- added J8: Conn_01x03_Male, symbol Connector:Conn_01x03_Male
- added R1: 160, Resistor_SMD:R_0805_2012Metric, symbol Device:R
- gave numbers to parts that had none: 30
Connections:
- net ECH0 is gone; now on net ECHO0: J9.1 (Pin_1)
- net +3.3V: now also J8.1 (Pin_1)
- net +5V: now also C1.1, D3.2 (A), J8.3 (Pin_3)
- net AMP1: now also J6.2 (Pin_2)
- net AMP2: now also J7.2 (Pin_2)
- net D25: now also J18.2 (Pin_2)
- net D26: now also J17.2 (Pin_2)
- net GND: now also C1.2, J6.1 (Pin_1), J7.1 (Pin_1), J8.2 (Pin_2), R1.2
- net L_TCRT: now also J18.1 (Pin_1)
- net R_TCRT: now also J17.1 (Pin_1)
- new net: D3.1 (K), R1.1
Other:
- note added: "Analógico"
- note added: "Comunicação placa de potência"
- note added: "Corrente Máx pin = 40mA"
- note added: "Divisor de tensão 3V"
- note added: "Placa possuí regulador interno de tensão"
- note added: "Sensor óptico"
- note added: "Tensão Máx pin = 3,3V"
- moved on the sheet: D4, D5, D6, J10, J15, J16, J19, J20, J21, J22, J3, J4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

Commit message: Update Shield_Esp32.kicad_sch
Parts:
- added C2: 100n, symbol Device:C
- added D7, D8: BAT54S, Package_TO_SOT_SMD:SOT-23, symbol Diode:BAT54S
- added J23: Conn_01x02_Male, Connector_PinHeader_2.54mm:PinHeader_1x02_P2.54mm_Vertical, symbol Connector:Conn_01x02_Male
- R2, R4: value 10k -> 15k
Connections:
- net +3.3V: now also C2.1, D7.2, D8.2
- net ADC2: now also D7.3, J23.1 (Pin_1)
- net ADC3: now also D8.3, J23.2 (Pin_2)
- net D13: now also J9.2 (Pin_2); no longer R2.2
- net D14: now also J15.2 (Pin_2); no longer R4.2
- net D25: now also R4.1
- net D26: now also R2.1
- net D32: now also D1.3, J1.2 (Pin_2)
- net D33: now also D2.3, J2.2 (Pin_2)
- net D34: no longer D1.3, J1.2 (Pin_2)
- net D35: no longer D2.3, J2.2 (Pin_2)
- net GND: now also R2.2, R4.2, C2.2, D7.1, D8.1
Other:
- note added: "Power"
- moved on the sheet: D1, D2, D5, D6, J1, J10, J11, J12, J13, J14, J15, J16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

Commit message: Inicio pcb
Parts:
- C1, C2: footprint (none) -> Capacitor_SMD:C_0805_2012Metric_Pad1.18x1.45mm_HandSolder
- D4: footprint (none) -> Diode_SMD:D_SMB
- J3: footprint (none) -> Connector_IDC:IDC-Header_2x13_P2.54mm_Vertical
- J4, J5: footprint (none) -> Connector_PinSocket_2.54mm:PinSocket_1x15_P2.54mm_Vertical
- J8: footprint (none) -> Connector_PinHeader_2.54mm:PinHeader_1x03_P2.54mm_Vertical
Connections:
- net D15: no longer J5.13 (Pin_13)
- net D23: no longer J5.1 (Pin_1)
- net D34: no longer J4.4 (Pin_4)
- net D35: no longer J4.5 (Pin_5)
- net D5: no longer J5.8 (Pin_8)
- net EN: no longer J4.1 (Pin_1)
- net RX2: no longer J5.10 (Pin_10)
- net TX2: no longer J5.9 (Pin_9)
- net VN: no longer J4.3 (Pin_3)
- net VP: no longer J4.2 (Pin_2)
- no-connect marks 1 -> 21

Commit message: pcb update
Parts:
- added H1, H2, H3: MountingHole, MountingHole:MountingHole_2.2mm_M2, symbol Mechanical:MountingHole
Changed lines of the file:
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@@
     (pin "1")
+  )
+  (symbol (lib_id "Mechanical:MountingHole") (at 266.7 161.29 0) (unit 1)
+    (in_bom yes) (on_board yes) (fields_autoplaced)
+    (property "Reference" "H3" (id 0) (at 269.24 160.0199 0)
+      (effects (font (size 1.27 1.27)) (justify left))
+    )
+    (property "Value" "MountingHole" (id 1) (at 269.24 162.5599 0)
+      (effects (font (size 1.27 1.27)) (justify left))
+    )
+    (property "Footprint" "MountingHole:MountingHole_2.2mm_M2" (id 2) (at 266.7 161.29 0)
+      (effects (font (size 1.27 1.27)) hide)
+    )
+    (property "Datasheet" "~" (id 3) (at 266.7 161.29 0)
+      (effects (font (size 1.27 1.27)) hide)
+    )
   )
   (symbol (lib_id "power:+3.3V") (at 39.37 90.17 0) (unit 1)
@@
     (property "Datasheet" "" (id 3) (at 119.38 53.34 0))
     (pin "1")
+  )
+  (symbol (lib_id "Mechanical:MountingHole") (at 266.7 156.21 0) (unit 1)
+    (in_bom yes) (on_board yes) (fields_autoplaced)
+    (property "Reference" "H2" (id 0) (at 269.24 154.9399 0)
+      (effects (font (size 1.27 1.27)) (justify left))
+    )
+    (property "Value" "MountingHole" (id 1) (at 269.24 157.4799 0)
+      (effects (font (size 1.27 1.27)) (justify left))
+    )
+    (property "Footprint" "MountingHole:MountingHole_2.2mm_M2" (id 2) (at 266.7 156.21 0)
+      (effects (font (size 1.27 1.27)) hide)
+    )
+    (property "Datasheet" "~" (id 3) (at 266.7 156.21 0)
+      (effects (font (size 1.27 1.27)) hide)
+    )
   )
   (symbol (lib_id "Connector:Conn_01x02_Male") (at 182.88 60.96 180) (unit 1)
@@
     (pin "2")
   )
+  (symbol (lib_id "Mechanical:MountingHole") (at 266.7 151.13 0) (unit 1)
+    (in_bom yes) (on_board yes) (fields_autoplaced)
+    (property "Reference" "H1" (id 0) (at 269.24 149.8599 0)
+      (effects (font (size 1.27 1.27)) (justify left))
+    )
+    (property "Value" "MountingHole" (id 1) (at 269.24 152.3999 0)
+      (effects (font (size 1.27 1.27)) (justify left))
+    )
+    (property "Footprint" "MountingHole:MountingHole_2.2mm_M2" (id 2) (at 266.7 151.13 0)
+      (effects (font (size 1.27 1.27)) hide)
+    )
+    (property "Datasheet" "~" (id 3) (at 266.7 151.13 0)
+      (effects (font (size 1.27 1.27)) hide)
+    )
+  )
   (sheet_instances
     (path "/" (page "1"))
@@
       (reference "D8") (unit 1) (value "BAT54S") (footprint "Package_TO_SOT_SMD:SOT-23")
     )
+    (path "/eedf7bc2-d18e-490b-92af-8529effa0518"
+      (reference "H1") (unit 1) (value "MountingHole") (footprint "MountingHole:MountingHole_2.2mm_M2")
+    )
+    (path "/cf60d3ac-cc16-4a11-a2a8-bda301aca295"
+      (reference "H2") (unit 1) (value "MountingHole") (footprint "MountingHole:MountingHole_2.2mm_M2")
+    )
+    (path "/a351814a-7d8f-4005-8f45-9a9d40b0a0ac"
+      (reference "H3") (unit 1) (value "MountingHole") (footprint "MountingHole:MountingHole_2.2mm_M2")
+    )
     (path "/2feeca62-2735-4a0e-bde4-e5e7203a9280"

Commit message: update pcb
Parts:
- added R10, R11: 10k, Resistor_SMD:R_0805_2012Metric, symbol Device:R
- R3, R5: value 15k -> 18,7k
Connections:
- net D13: now also R10.2; no longer J9.2 (Pin_2)
- net D14: now also R11.2; no longer J15.2 (Pin_2)
- new net: J9.2 (Pin_2), R10.1
- new net: J15.2 (Pin_2), R11.1
Other:
- moved on the sheet: J15, J16, R3, R5

Commit message: update encoder
Parts:
- R8, R9: value 15k -> 20k
Changed lines of the file:
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@@
       (effects (font (size 1.27 1.27)) (justify left))
     )
-    (property "Value" "15k" (id 1) (at 127.508 175.133 0)
+    (property "Value" "20k" (id 1) (at 127.508 175.133 0)
       (effects (font (size 1.27 1.27)) (justify left))
     )
@@
       (effects (font (size 1.27 1.27)) (justify left))
     )
-    (property "Value" "15k" (id 1) (at 165.608 175.133 0)
+    (property "Value" "20k" (id 1) (at 165.608 175.133 0)
       (effects (font (size 1.27 1.27)) (justify left))
     )
@@
     )
     (path "/8cc10a9a-2477-4232-996c-c25bf899d45f"
-      (reference "R8") (unit 1) (value "15k") (footprint "Resistor_SMD:R_0805_2012Metric")
+      (reference "R8") (unit 1) (value "20k") (footprint "Resistor_SMD:R_0805_2012Metric")
     )
     (path "/9050431d-caa7-4f21-aaf0-07d9d33e1446"
-      (reference "R9") (unit 1) (value "15k") (footprint "Resistor_SMD:R_0805_2012Metric")
+      (reference "R9") (unit 1) (value "20k") (footprint "Resistor_SMD:R_0805_2012Metric")
     )
     (path "/6ba7466b-3e6d-4a1a-bec1-33e4e97e49b6"
